Commit message: Update stretch.urdf

File: resource/urdf/stretch/stretch.urdf (robot description, URDF)
Before this commit: robot stretch, 20 links, 19 joints
Links:
- added link virtual_link_x
- added link world_base
- added link world_base_z_lift
Joints:
- added joint base_prismatic_joint_x: type prismatic, parent virtual_link_x, child base_link, origin xyz=0 0 0 rpy=0 0 0, axis 1 0 0, limit lower=-200.0 upper=200.0 effort=1000 velocity=1.0
- added joint base_rotation_joint: type continuous, parent world_base_z_lift, child virtual_link_x, origin xyz=0 0 0 rpy=0 0 0, axis 0 0 1
- added joint z_lift_fixed_joint: type fixed, parent world_base, child world_base_z_lift, origin xyz=0 0 0.005 rpy=0 0 0

Commit message: Revert "Update main repo changes"

File: resource/urdf/stretch/stretch.urdf (robot description, URDF)
Before this commit: robot stretch, 23 links, 22 joints
Links:
- removed link virtual_link_x
- removed link world_base
- removed link world_base_z_lift
Joints:
- removed joint base_prismatic_joint_x
- removed joint base_rotation_joint
- removed joint z_lift_fixed_joint

Commit message: add plate to robot and commet out walls and floating cabinet

File: resource/urdf/stretch/stretch.urdf (robot description, URDF)
Before this commit: robot stretch, 20 links, 19 joints
Links:
- added link plate, mass 1.0; collision box size=0.4 0.4 0.02; visual box size=0.4 0.4 0.02
Joints:
- added joint plate_joint: type fixed, parent base_link, child plate, origin xyz=0 0 0.2 rpy=0 0 0

Commit message: fix coordination system problem

File: resource/urdf/stretch/stretch.urdf (robot description, URDF)
Before this commit: robot stretch, 23 links, 22 joints
Links:
- added link virtual_link_y
Joints:
- added joint base_prismatic_joint_y: type prismatic, parent virtual_link_x, child virtual_link_y, origin xyz=0 0 0 rpy=0 0 0, axis 0 1 0, limit lower=-200.0 upper=200.0 effort=1000 velocity=1.0
- joint base_prismatic_joint_x: child base_link -> virtual_link_x; parent virtual_link_x -> world_base_z_lift
- joint base_rotation_joint: child virtual_link_x -> base_link; parent world_base_z_lift -> virtual_link_y

Commit message: fix everything

File: resource/urdf/stretch/stretch.urdf (robot description, URDF)
Before this commit: robot stretch, 24 links, 23 joints
Joints:
- joint joint_left_finger: limit lower=-0.05 upper=0.0 effort=100 velocity=1.0 -> lower=-0.03 upper=0.02 effort=100 velocity=1.0
- joint joint_right_finger: limit lower=0 upper=0.05 effort=100 velocity=1.0 -> lower=-0.02 upper=0.03 effort=100 velocity=1.0
